File: solid_state_relays_24v.kicad_pcb (KiCad board)
At the start: 2 copper layers, 120 x 90 mm, 68 parts, among them J1 1190297, J2 1190297, J3 1190297, J4 1190297, J5 1190297, J6 1190297, J7 1190297, J8 1190297, Q1 IRF4905PBF, Q2 IRF4905PBF, Q3 IRF4905PBF, Q4 IRF4905PBF, Q5 IRF4905PBF, Q6 IRF4905PBF, Q7 IRF4905PBF, Q8 IRF4905PBF

Commit message: Admin updates to v0.0.6
Other:
- board text added: "Rev: 0.0.6"
Changed lines of the file:
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@@
   )
   (layers
-    (0 "F.Cu" signal)
-    (31 "B.Cu" signal)
+    (0 "F.Cu" mixed)
+    (31 "B.Cu" mixed)
     (32 "B.Adhes" user "B.Adhesive")
     (33 "F.Adhes" user "F.Adhesive")
@@
   (setup
     (stackup
-      (layer "F.SilkS" (type "Top Silk Screen") (color "White"))
+      (layer "F.SilkS" (type "Top Silk Screen") (color "White") (material "Liquid Photo"))
       (layer "F.Paste" (type "Top Solder Paste"))
-      (layer "F.Mask" (type "Top Solder Mask") (color "Red") (thickness 0.01))
+      (layer "F.Mask" (type "Top Solder Mask") (color "Red") (thickness 0.01) (material "Liquid Ink") (epsilon_r 3.3) (loss_tangent 0))
       (layer "F.Cu" (type "copper") (thickness 0.07))
       (layer "dielectric 1" (type "core") (thickness 1.6) (material "FR4") (epsilon_r 4.5) (loss_tangent 0.02))
       (layer "B.Cu" (type "copper") (thickness 0.07))
-      (layer "B.Mask" (type "Bottom Solder Mask") (color "Red") (thickness 0.01))
+      (layer "B.Mask" (type "Bottom Solder Mask") (color "Red") (thickness 0.01) (material "Liquid Ink") (epsilon_r 3.3) (loss_tangent 0))
       (layer "B.Paste" (type "Bottom Solder Paste"))
-      (layer "B.SilkS" (type "Bottom Silk Screen") (color "White"))
+      (layer "B.SilkS" (type "Bottom Silk Screen") (color "White") (material "Liquid Photo"))
       (copper_finish "HAL lead-free")
       (dielectric_constraints no)
@@
   )
   (gr_rect (start 50 50) (end 170 140) (layer "Edge.Cuts") (width 0.001) (fill none))
+  (gr_text "Rev: 0.0.6" (at 110 101) (layer "F.SilkS")
+    (effects (font (size 2 2) (thickness 0.5)))
+  )
   (gr_text "1.7600 mm" (at 144.348571 179.13) (layer "User.2")
     (effects (font (size 1.5 1.5) (thickness 0.2)) (justify left top))

Commit message: Updating schematic and PCB for v0.0.8
Parts:
- added TVSP1: SM6T30AY, dragon_mobile:SMBJ36CATR, F.Cu at (70.2, 95.0)
- J1, J2, J3, J4, J5, J6, J7, J8: footprint Connector_Pheonix_Other:1190297 -> dragon_mobile:1190297
- JPWR1: footprint Dragon:Amass_XT60PW-M_Kombifootprint -> dragon_mobile:Amass_XT60PW-M_Kombifootprint
- LED1, LED2, LED3, LED4, LED5, LED6, LED7, LED8: value (red) -> LTST-C190KFKT; footprint SamacSys_Parts:LEDC2012X120N -> dragon_mobile:LEDC1607X80N
- LEDP1: value (red) -> LTST-C190KGKT; footprint SamacSys_Parts:LEDC2012X120N -> dragon_mobile:LEDC1608X80N
- Q1, Q2, Q3, Q4, Q5, Q6, Q7, Q8: footprint SamacSys_Parts:TO254P469X1042X1967-3P -> dragon_mobile:TO254P469X1042X1967-3P
- R1: value 1.2k -> 1k2; footprint Resistor_SMD:R_0805_2012Metric -> Resistor_SMD:R_0603_1608Metric_Pad0.98x0.95mm_HandSolder
- RL1, RL2, RL3, RL4, RL5, RL6, RL7, RL8: value 1.2k -> 1k2
- TVS1, TVS2, TVS3, TVS4, TVS5, TVS6, TVS7, TVS8: value SM6T30A -> SM6T30AY; footprint Diode_SMD:D_SMB -> dragon_mobile:SMBJ36CATR
- moved TVS1 19.0 mm to (57.5, 67.0)
- moved TVS2 19.0 mm to (82.5, 67.0)
- moved TVS3 19.0 mm to (107.5, 67.0)
- moved TVS4 19.0 mm to (132.5, 67.0)
- moved TVS5 19.0 mm to (162.5, 123.0)
- moved TVS6 19.0 mm to (137.5, 123.0)
- moved TVS7 19.0 mm to (112.5, 123.0)
- moved TVS8 19.0 mm to (87.5, 123.0)
- moved #LOGO1 2.50 mm to (97.5, 95.0)
- moved #LOGO2 2.50 mm to (82.5, 95.0)
- moved LED1 1.35 mm to (75.2, 53.5)
- moved LED2 1.35 mm to (100.2, 53.5)
- moved LED3 1.35 mm to (125.2, 53.5)
- moved LED4 1.35 mm to (150.2, 53.5)
- moved LED5 1.35 mm to (144.8, 136.5)
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Connections:
- HC1 pad 1: (no net) -> GNDPWR
- R1 pad 1: +BATT -> Net-(LEDP1-Pad2)
- R1 pad 2: Net-(LEDP1-Pad2) -> +BATT
- RL1 pad 1: Net-(LED1-Pad2) -> OUT1
- RL1 pad 2: OUT1 -> Net-(LED1-Pad2)
- RL2 pad 1: Net-(LED2-Pad2) -> OUT2
- RL2 pad 2: OUT2 -> Net-(LED2-Pad2)
- RL3 pad 1: Net-(LED3-Pad2) -> OUT3
- RL3 pad 2: OUT3 -> Net-(LED3-Pad2)
- RL4 pad 1: Net-(LED4-Pad2) -> OUT4
- RL4 pad 2: OUT4 -> Net-(LED4-Pad2)
- RL5 pad 1: Net-(LED5-Pad2) -> OUT5
- RL5 pad 2: OUT5 -> Net-(LED5-Pad2)
- RL6 pad 1: Net-(LED6-Pad2) -> OUT6
- RL6 pad 2: OUT6 -> Net-(LED6-Pad2)
- RL7 pad 1: Net-(LED7-Pad2) -> OUT7
- RL7 pad 2: OUT7 -> Net-(LED7-Pad2)
- RL8 pad 1: Net-(LED8-Pad2) -> OUT8
- RL8 pad 2: OUT8 -> Net-(LED8-Pad2)
- RP1 pad 1: +BATT -> /a1
- RP1 pad 2: /a1 -> +BATT
- RP2 pad 1: +BATT -> /a2
- RP2 pad 2: /a2 -> +BATT
- RP3 pad 1: +BATT -> /a3
- RP3 pad 2: /a3 -> +BATT
- RP4 pad 1: +BATT -> /a4
- RP4 pad 2: /a4 -> +BATT
- RP5 pad 1: +BATT -> /a5
- RP5 pad 2: /a5 -> +BATT
- RP6 pad 1: +BATT -> /a6
- RP6 pad 2: /a6 -> +BATT
- RP7 pad 1: +BATT -> /a7
- RP7 pad 2: /a7 -> +BATT
- RP8 pad 1: +BATT -> /a8
- RP8 pad 2: /a8 -> +BATT
Routing:
- net +BATT: track 454.3 -> 531.0 mm, vias 16 -> 70
- net GNDPWR: track 7.96 -> 5.33 mm, vias 31 -> 107
Other:
- board text added: "+"
- board text added: "Rev: 0.0.8"
- board text removed: "Rev: 0.0.6"

Commit message: v0.0.10-pre2
Parts:
- added JP1: SolderJumper_2_Bridged, Jumper:SolderJumper-2_P1.3mm_Bridged_RoundedPad1.0x1.5mm, F.Cu at (63.5, 67.8)
- added TVSP2: SM6T30AY, dragon_mobile:SMBJ36CATR, F.Cu at (55.2, 83.3)
- JPWR1: value XT60PW-M_Kombifootprint -> XT60PW-M; footprint dragon_mobile:Amass_XT60PW-M_Kombifootprint -> dragon_mobile:XT60PWM
- R1: value 1k2 -> 1k5; footprint Resistor_SMD:R_0603_1608Metric_Pad0.98x0.95mm_HandSolder -> dragon_mobile:RESC2012X65N
- RL1, RL2, RL3, RL4, RL5, RL6, RL7, RL8: value 1k2 -> 1k5; footprint Resistor_SMD:R_0805_2012Metric -> dragon_mobile:RESC2012X65N
- RP1, RP2, RP3, RP4, RP5, RP6, RP7, RP8: footprint Resistor_SMD:R_0805_2012Metric -> dragon_mobile:RESC2012X65N
- moved LEDP1 41.0 mm to (57.5, 64.0)
- moved R1 41.0 mm to (62.5, 64.0)
- moved TVS1 25.5 mm to (83.0, 68.2)
- moved TVS2 25.5 mm to (108.0, 68.2)
- moved TVS3 25.5 mm to (133.0, 68.2)
- moved TVS4 25.5 mm to (158.0, 68.2)
- moved TVS5 25.5 mm to (137.0, 121.8)
- moved TVS6 25.5 mm to (112.0, 121.8)
- moved TVS7 25.5 mm to (87.0, 121.8)
- moved TVS8 25.5 mm to (62.0, 121.8)
- moved HQ1 21.0 mm to (60.2, 77.5)
- moved HQ2 21.0 mm to (85.2, 77.5)
- moved HQ3 21.0 mm to (110.2, 77.5)
- moved HQ4 21.0 mm to (135.2, 77.5)
- moved HQ5 21.0 mm to (159.8, 112.5)
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Connections:
- R1 pad 2: +BATT -> Net-(JP1-Pad2)
Routing:
- net +BATT: track 531.0 -> 11.7 mm, vias 70 -> 99
- net OUT3: track 55.9 -> 70.2 mm, vias 0 -> 7
- net OUT2: track 55.9 -> 70.2 mm, vias 0 -> 7
- net OUT1: track 55.9 -> 70.2 mm, vias 0 -> 7
- net OUT8: track 55.9 -> 70.2 mm, vias 0 -> 7
- net OUT7: track 55.9 -> 70.2 mm, vias 0 -> 7
- net OUT6: track 55.9 -> 70.2 mm, vias 0 -> 7
- net OUT4: track 55.9 -> 70.2 mm, vias 0 -> 7
- net OUT5: track 55.9 -> 70.2 mm, vias 0 -> 7
- net /a7: track 59.8 -> 73.3 mm
- net /a6: track 31.2 -> 44.7 mm
- net /a8: track 82.3 -> 95.8 mm
- net /a3: track 45.2 -> 36.5 mm
- net /a2: track 73.9 -> 65.2 mm
- net /a1: track 96.3 -> 87.7 mm
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Other:
- board text added: "Rev: 0.0.10"
- board text added: "https://github.com/dragon-mobile/solid_state_relays_24v"
- board text added: "© 2022 Michael Cummings"
- board text removed: "Rev: 0.0.8"

Commit message: WIP
Parts:
- renumbered HQ4 to HQ1, HQ3 to HQ2, HQ2 to HQ3, HQ1 to HQ4, HQ8 to HQ5, HQ7 to HQ6, HQ6 to HQ7, HQ5 to HQ8, J4 to J1, J3 to J2, J2 to J3, J1 to J4, J8 to J5, J7 to J6, J6 to J7, J5 to J8, LED4 to LED1, LED3 to LED2, LED2 to LED3, LED1 to LED4, LED8 to LED5, LED7 to LED6, LED6 to LED7, LED5 to LED8, Q4 to Q1, Q3 to Q2, Q2 to Q3, Q1 to Q4, Q8 to Q5, Q7 to Q6, Q6 to Q7, Q5 to Q8, RL4 to RL1, RL3 to RL2, RL2 to RL3, RL1 to RL4, RL8 to RL5, RL7 to RL6, RL6 to RL7, RL5 to RL8, RP4 to RP1, RP3 to RP2, RP2 to RP3, RP1 to RP4, RP8 to RP5, RP7 to RP6, RP6 to RP7, RP5 to RP8, TVS4 to TVS1, TVS3 to TVS2, TVS2 to TVS3, TVS1 to TVS4, TVS8 to TVS5, TVS7 to TVS6, TVS6 to TVS7, TVS5 to TVS8
Connections:
- J1 pad 1: OUT4 -> OUT1
- J1 pad 2: OUT4 -> OUT1
- J1 pad 3: OUT4 -> OUT1
- J1 pad 4: OUT4 -> OUT1
- J2 pad 1: OUT3 -> OUT2
- J2 pad 2: OUT3 -> OUT2
- J2 pad 3: OUT3 -> OUT2
- J2 pad 4: OUT3 -> OUT2
- J3 pad 1: OUT2 -> OUT3
- J3 pad 2: OUT2 -> OUT3
- J3 pad 3: OUT2 -> OUT3
- J3 pad 4: OUT2 -> OUT3
- J4 pad 1: OUT1 -> OUT4
- J4 pad 2: OUT1 -> OUT4
- J4 pad 3: OUT1 -> OUT4
- J4 pad 4: OUT1 -> OUT4
- J5 pad 1: OUT8 -> OUT5
- J5 pad 2: OUT8 -> OUT5
- J5 pad 3: OUT8 -> OUT5
- J5 pad 4: OUT8 -> OUT5
- J6 pad 1: OUT7 -> OUT6
- J6 pad 2: OUT7 -> OUT6
- J6 pad 3: OUT7 -> OUT6
- J6 pad 4: OUT7 -> OUT6
- J7 pad 1: OUT6 -> OUT7
- J7 pad 2: OUT6 -> OUT7
- J7 pad 3: OUT6 -> OUT7
- J7 pad 4: OUT6 -> OUT7
- J8 pad 1: OUT5 -> OUT8
- J8 pad 2: OUT5 -> OUT8
- J8 pad 3: OUT5 -> OUT8
- J8 pad 4: OUT5 -> OUT8
- JCNTL1 pad 10: /a5 -> /a8
- JCNTL1 pad 3: /a3 -> /a2
- JCNTL1 pad 4: /a4 -> /a1
- JCNTL1 pad 5: /a1 -> /a4
- JCNTL1 pad 6: /a2 -> /a3
- JCNTL1 pad 7: /a8 -> /a5
- JCNTL1 pad 8: /a7 -> /a6
- JCNTL1 pad 9: /a6 -> /a7
- Q1 pad 1: /a4 -> /a1
- Q1 pad 3: OUT4 -> OUT1
- Q2 pad 1: /a3 -> /a2
- Q2 pad 3: OUT3 -> OUT2
- Q3 pad 1: /a2 -> /a3
- Q3 pad 3: OUT2 -> OUT3
- Q4 pad 1: /a1 -> /a4
- Q4 pad 3: OUT1 -> OUT4
- Q5 pad 1: /a8 -> /a5
- Q5 pad 3: OUT8 -> OUT5
- Q6 pad 1: /a7 -> /a6
- Q6 pad 3: OUT7 -> OUT6
- Q7 pad 1: /a6 -> /a7
- Q7 pad 3: OUT6 -> OUT7
- Q8 pad 1: /a5 -> /a8
- Q8 pad 3: OUT5 -> OUT8
- RL1 pad 1: OUT4 -> OUT1
- RL2 pad 1: OUT3 -> OUT2
- RL3 pad 1: OUT2 -> OUT3
- RL4 pad 1: OUT1 -> OUT4
- RL5 pad 1: OUT8 -> OUT5
- RL6 pad 1: OUT7 -> OUT6
- RL7 pad 1: OUT6 -> OUT7
- RL8 pad 1: OUT5 -> OUT8
- RP1 pad 1: /a4 -> /a1
- RP2 pad 1: /a3 -> /a2
- RP3 pad 1: /a2 -> /a3
- RP4 pad 1: /a1 -> /a4
- RP5 pad 1: /a8 -> /a5
- RP6 pad 1: /a7 -> /a6
- RP7 pad 1: /a6 -> /a7
- RP8 pad 1: /a5 -> /a8
- TVS1 pad 2: OUT4 -> OUT1
- TVS2 pad 2: OUT3 -> OUT2
- TVS3 pad 2: OUT2 -> OUT3
- TVS4 pad 2: OUT1 -> OUT4
- TVS5 pad 2: OUT8 -> OUT5
- TVS6 pad 2: OUT7 -> OUT6
- TVS7 pad 2: OUT6 -> OUT7
- TVS8 pad 2: OUT5 -> OUT8
Routing:
- net /a8: track 95.8 -> 22.2 mm
- net /a5: track 22.2 -> 95.8 mm
- net /a4: track 15.3 -> 87.7 mm
- net /a1: track 87.7 -> 15.3 mm
- net /a3: track 36.5 -> 65.2 mm
- net /a2: track 65.2 -> 36.5 mm
- net /a7: track 73.3 -> 44.7 mm
- net /a6: track 44.7 -> 73.3 mm
